File: DRV_motordriver/DRV_motor_driver.kicad_sch (KiCad schematic)
At the start: 35 parts, among them J1 jumper, J2 jumper, J3 Conn_01x02, J4 Conn_01x02, J5 Conn_01x02, J6 Conn_01x02, J7 Conn_01x02, Q1 NMOS, Q2 NMOS, Q3 NMOS, Q4 NMOS, Q5 NMOS, Q6 NMOS, Q7 NMOS, Q8 NMOS, U1 DRV8701PRGER, U2 DRV8701PRGER

Commit message: update library for DRV_motor_driver
Parts:
- C1, C10, C11, C2, C3, C4, C5, C6, C7, C8, C9: symbol HKUST_RDC2025_Symbol_Lib:C_Small -> DRV_motor_driver:C_Small
- D1, D2: symbol HKUST_RDC2025_Symbol_Lib:SS54 -> DRV_motor_driver:SS54
- H1, H2, H3, H4: symbol HKUST_RDC2024_Symbol_Lib:MountingHole -> DRV_motor_driver:MountingHole
- J1, J2: symbol Connector_Generic:Conn_01x03 -> DRV_motor_driver:Conn_01x03
- J3, J4, J5, J6, J7: symbol Connector_Generic:Conn_01x02 -> DRV_motor_driver:Conn_01x02
- Q1, Q2, Q3, Q4, Q5, Q6, Q7, Q8: symbol Simulation_SPICE:NMOS -> DRV_motor_driver:NMOS
- S1: symbol STC8H&16F&32G_主板_V3.1:SW-SPDT -> DRV_motor_driver:SW-SPDT
- U1, U2: symbol DRV8701PRGER:DRV8701PRGER -> DRV_motor_driver:DRV8701PRGER
Changed lines of the file:
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@@
 	)
 	(symbol
-		(lib_id "Simulation_SPICE:NMOS")
+		(lib_id "DRV_motor_driver:NMOS")
 		(at 194.31 158.75 0)
 		(unit 1)
@@
 	)
 	(symbol
-		(lib_id "Simulation_SPICE:NMOS")
+		(lib_id "DRV_motor_driver:NMOS")
 		(at 226.06 73.66 0)
 		(unit 1)
@@
 	)
 	(symbol
-		(lib_id "DRV8701PRGER:DRV8701PRGER")
+		(lib_id "DRV_motor_driver:DRV8701PRGER")
 		(at 105.41 88.9 0)
 		(unit 1)
@@
 	)
 	(symbol
-		(lib_id "HKUST_RDC2025_Symbol_Lib:C_Small")
+		(lib_id "DRV_motor_driver:C_Small")
 		(at 158.75 161.29 0)
 		(unit 1)
@@
 	)
 	(symbol
-		(lib_id "HKUST_RDC2025_Symbol_Lib:C_Small")
+		(lib_id "DRV_motor_driver:C_Small")
 		(at 133.35 158.75 0)
 		(unit 1)
@@
 	)
 	(symbol
-		(lib_id "Connector_Generic:Conn_01x02")
+		(lib_id "DRV_motor_driver:Conn_01x02")
 		(at 267.97 88.9 0)
 		(unit 1)
@@
 	)
 	(symbol
-		(lib_id "Simulation_SPICE:NMOS")
+		(lib_id "DRV_motor_driver:NMOS")
 		(at 194.31 53.34 0)
 		(unit 1)
@@
 	)
 	(symbol
-		(lib_id "STC8H&16F&32G_主板_V3.1:SW-SPDT")
+		(lib_id "DRV_motor_driver:SW-SPDT")
 		(at 265.43 128.27 0)
 		(unit 1)
@@
 	)
 	(symbol
-		(lib_id "Simulation_SPICE:NMOS")
+		(lib_id "DRV_motor_driver:NMOS")
 		(at 226.06 158.75 0)
 		(unit 1)
@@
 	)
 	(symbol
-		(lib_id "HKUST_RDC2025_Symbol_Lib:C_Small")
+		(lib_id "DRV_motor_driver:C_Small")
 		(at 140.97 68.58 270)
 		(unit 1)
@@
 	)
 	(symbol
-		(lib_id "HKUST_RDC2025_Symbol_Lib:C_Small")
+		(lib_id "DRV_motor_driver:C_Small")
 		(at 125.73 135.89 90)
 		(unit 1)
@@
 	)
 	(symbol
-		(lib_id "HKUST_RDC2025_Symbol_Lib:C_Small")
+		(lib_id "DRV_motor_driver:C_Small")
 		(at 129.54 50.8 90)
 		(unit 1)
@@
 	)
 	(symbol
-		(lib_id "HKUST_RDC2024_Symbol_Lib:MountingHole")
+		(lib_id "DRV_motor_driver:MountingHole")
 		(at 212.09 631.19 0)
 		(unit 1)
@@
 	)
 	(symbol
-		(lib_id "HKUST_RDC2024_Symbol_Lib:MountingHole")
+		(lib_id "DRV_motor_driver:MountingHole")
 		(at 185.42 640.08 0)
 		(unit 1)
@@
 	)
 	(symbol
-		(lib_id "Connector_Generic:Conn_01x02")
+		(lib_id "DRV_motor_driver:Conn_01x02")
 		(at 267.97 93.98 0)
 		(unit 1)
@@
 	)
 	(symbol
-		(lib_id "HKUST_RDC2024_Symbol_Lib:MountingHole")
+		(lib_id "DRV_motor_driver:MountingHole")
 		(at 185.42 631.19 0)
 		(unit 1)
@@
 	)
 	(symbol
-		(lib_id "HKUST_RDC2025_Symbol_Lib:C_Small")
+		(lib_id "DRV_motor_driver:C_Small")
 		(at 321.31 129.54 0)
 		(unit 1)
@@
 	)
 	(symbol
-		(lib_id "HKUST_RDC2025_Symbol_Lib:SS54")
+		(lib_id "DRV_motor_driver:SS54")
 		(at 163.83 153.67 0)
 		(unit 1)
@@
 	)
 	(symbol
-		(lib_id "HKUST_RDC2025_Symbol_Lib:C_Small")
+		(lib_id "DRV_motor_driver:C_Small")
 		(at 147.32 161.29 0)
 		(unit 1)
@@
 	)
 	(symbol
-		(lib_id "Connector_Generic:Conn_01x02")
+		(lib_id "DRV_motor_driver:Conn_01x02")
 		(at 267.97 110.49 0)
 		(unit 1)
@@
 	)
 	(symbol
-		(lib_id "HKUST_RDC2025_Symbol_Lib:SS54")
+		(lib_id "DRV_motor_driver:SS54")
 		(at 163.83 68.58 0)
 		(unit 1)
@@
 	)
 	(symbol
-		(lib_id "HKUST_RDC2025_Symbol_Lib:C_Small")
+		(lib_id "DRV_motor_driver:C_Small")
 		(at 133.35 73.66 0)
 		(unit 1)
@@
 	)
 	(symbol
-		(lib_id "Connector_Generic:Conn_01x02")
+		(lib_id "DRV_motor_driver:Conn_01x02")
 		(at 267.97 105.41 0)
 		(unit 1)
@@
 	)
 	(symbol
-		(lib_id "Simulation_SPICE:NMOS")
+		(lib_id "DRV_motor_driver:NMOS")
 		(at 194.31 73.66 0)
 		(unit 1)
@@
 	)
 	(symbol
-		(lib_id "Simulation_SPICE:NMOS")
+		(lib_id "DRV_motor_driver:NMOS")
 		(at 226.06 53.34 0)
 		(unit 1)
@@
 	)
 	(symbol
-		(lib_id "Connector_Generic:Conn_01x02")
+		(lib_id "DRV_motor_driver:Conn_01x02")
 		(at 284.48 128.27 0)
 		(unit 1)
@@
 	)
 	(symbol
-		(lib_id "Simulation_SPICE:NMOS")
+		(lib_id "DRV_motor_driver:NMOS")
 		(at 194.31 138.43 0)
 		(unit 1)
@@
 	)
 	(symbol
-		(lib_id "Connector_Generic:Conn_01x03")
+		(lib_id "DRV_motor_driver:Conn_01x03")
 		(at 53.34 83.82 180)
 		(unit 1)
@@
 	)
 	(symbol
-		(lib_id "HKUST_RDC2025_Symbol_Lib:C_Small")
+		(lib_id "DRV_motor_driver:C_Small")
 		(at 147.32 76.2 0)
 		(unit 1)
@@
 	)
 	(symbol
-		(lib_id "HKUST_RDC2025_Symbol_Lib:C_Small")
+		(lib_id "DRV_motor_driver:C_Small")
 		(at 140.97 153.67 270)
 		(unit 1)
@@
 	)
 	(symbol
-		(lib_id "DRV8701PRGER:DRV8701PRGER")
+		(lib_id "DRV_motor_driver:DRV8701PRGER")
 		(at 105.41 173.99 0)
 		(unit 1)
@@
 	)
 	(symbol
-		(lib_id "Simulation_SPICE:NMOS")
+		(lib_id "DRV_motor_driver:NMOS")
 		(at 226.06 138.43 0)
 		(unit 1)
@@
 	)
 	(symbol
-		(lib_id "HKUST_RDC2024_Symbol_Lib:MountingHole")
+		(lib_id "DRV_motor_driver:MountingHole")
 		(at 212.09 641.35 0)
 		(unit 1)
@@
 	)
 	(symbol
-		(lib_id "Connector_Generic:Conn_01x03")
+		(lib_id "DRV_motor_driver:Conn_01x03")
 		(at 53.34 168.91 180)
 		(unit 1)
@@
 	)
 	(symbol
-		(lib_id "HKUST_RDC2025_Symbol_Lib:C_Small")
+		(lib_id "DRV_motor_driver:C_Small")
 		(at 158.75 76.2 0)
 		(unit 1)
