File: sensor_board/sensor_board.kicad_pcb (KiCad board)
At the start: 2 copper layers, 68.8 x 40 mm, 24 parts, among them J2 FFC2A32-10-T, U1 QRE1113GR, U2 QRE1113GR, U3 QRE1113GR, U4 QRE1113GR, U5 QRE1113GR, U6 QRE1113GR, U7 QRE1113GR

Commit message: update lib and step for sensor board
Parts:
- H1, H2: footprint HKUST_RDC2024_Footprint_Lib:MountingHole_3.2mm_M3 -> forklift_sensor_board:MountingHole_3.2mm_M3
- J2: footprint FFC2A32-10-T:GCT_FFC2A32-10-T -> forklift_sensor_board:GCT_FFC2A32-10-T
- R1, R10, R11, R12, R13, R14, R2, R3, R4, R5, R6, R7, R8, R9: footprint HKUST_RDC2024_Footprint_Lib:R_0603_1608Metric -> forklift_sensor_board:R_0603_1608Metric
- U1, U2, U3, U4, U5, U6, U7: footprint OptoDevice:OnSemi_CASE100CY -> forklift_sensor_board:OnSemi_CASE100CY
Changed lines of the file:
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@@
 	(net 19 "unconnected-(J2-SHIELD-PadS1)_2")
 	(net 20 "unconnected-(J2-SHIELD-PadS1)_3")
-	(footprint "OptoDevice:OnSemi_CASE100CY"
+	(footprint "forklift_sensor_board:OnSemi_CASE100CY"
 		(layer "F.Cu")
 		(at 80.567 138.297)
@@
 		)
 	)
-	(footprint "HKUST_RDC2024_Footprint_Lib:R_0603_1608Metric"
+	(footprint "forklift_sensor_board:R_0603_1608Metric"
 		(layer "F.Cu")
 		(at 108.95 132.716 -90)
@@
 		)
 	)
-	(footprint "HKUST_RDC2024_Footprint_Lib:R_0603_1608Metric"
+	(footprint "forklift_sensor_board:R_0603_1608Metric"
 		(layer "F.Cu")
 		(at 89.427 132.747 -90)
@@
 		)
 	)
-	(footprint "HKUST_RDC2024_Footprint_Lib:R_0603_1608Metric"
+	(footprint "forklift_sensor_board:R_0603_1608Metric"
 		(layer "F.Cu")
 		(at 79.615 132.714 -90)
@@
 		)
 	)
-	(footprint "HKUST_RDC2024_Footprint_Lib:R_0603_1608Metric"
+	(footprint "forklift_sensor_board:R_0603_1608Metric"
 		(layer "F.Cu")
 		(at 80.517 129.834)
@@
 		)
 	)
-	(footprint "HKUST_RDC2024_Footprint_Lib:R_0603_1608Metric"
+	(footprint "forklift_sensor_board:R_0603_1608Metric"
 		(layer "F.Cu")
 		(at 100.041 129.834)
@@
 		)
 	)
-	(footprint "OptoDevice:OnSemi_CASE100CY"
+	(footprint "forklift_sensor_board:OnSemi_CASE100CY"
 		(layer "F.Cu")
 		(at 70.805 138.297)
@@
 		)
 	)
-	(footprint "HKUST_RDC2024_Footprint_Lib:R_0603_1608Metric"
+	(footprint "forklift_sensor_board:R_0603_1608Metric"
 		(layer "F.Cu")
 		(at 119.565 129.834)
@@
 		)
 	)
-	(footprint "HKUST_RDC2024_Footprint_Lib:R_0603_1608Metric"
+	(footprint "forklift_sensor_board:R_0603_1608Metric"
 		(layer "F.Cu")
 		(at 69.936 132.648 -90)
@@
 		)
 	)
-	(footprint "HKUST_RDC2024_Footprint_Lib:MountingHole_3.2mm_M3"
+	(footprint "forklift_sensor_board:MountingHole_3.2mm_M3"
 		(layer "F.Cu")
 		(at 121.43 111.483)
@@
 		)
 	)
-	(footprint "OptoDevice:OnSemi_CASE100CY"
+	(footprint "forklift_sensor_board:OnSemi_CASE100CY"
 		(layer "F.Cu")
 		(at 90.2915 138.297)
@@
 		)
 	)
-	(footprint "HKUST_RDC2024_Footprint_Lib:R_0603_1608Metric"
+	(footprint "forklift_sensor_board:R_0603_1608Metric"
 		(layer "F.Cu")
 		(at 70.755 129.834)
@@
 		)
 	)
-	(footprint "HKUST_RDC2024_Footprint_Lib:R_0603_1608Metric"
+	(footprint "forklift_sensor_board:R_0603_1608Metric"
 		(layer "F.Cu")
 		(at 128.474 132.731 -90)
@@
 		)
 	)
-	(footprint "HKUST_RDC2024_Footprint_Lib:R_0603_1608Metric"
+	(footprint "forklift_sensor_board:R_0603_1608Metric"
 		(layer "F.Cu")
 		(at 118.661 132.78 -90)
@@
 		)
 	)
-	(footprint "HKUST_RDC2024_Footprint_Lib:R_0603_1608Metric"
+	(footprint "forklift_sensor_board:R_0603_1608Metric"
 		(layer "F.Cu")
 		(at 90.279 129.834)
@@
 		)
 	)
-	(footprint "OptoDevice:OnSemi_CASE100CY"
+	(footprint "forklift_sensor_board:OnSemi_CASE100CY"
 		(layer "F.Cu")
 		(at 129.302 138.297)
@@
 		)
 	)
-	(footprint "HKUST_RDC2024_Footprint_Lib:R_0603_1608Metric"
+	(footprint "forklift_sensor_board:R_0603_1608Metric"
 		(layer "F.Cu")
 		(at 109.803 129.834)
@@
 		)
 	)
-	(footprint "HKUST_RDC2024_Footprint_Lib:R_0603_1608Metric"
+	(footprint "forklift_sensor_board:R_0603_1608Metric"
 		(layer "F.Cu")
 		(at 129.327 129.834)
@@
 		)
 	)
-	(footprint "HKUST_RDC2024_Footprint_Lib:MountingHole_3.2mm_M3"
+	(footprint "forklift_sensor_board:MountingHole_3.2mm_M3"
 		(layer "F.Cu")
 		(at 78.445 111.483)
@@
 		)
 	)
-	(footprint "OptoDevice:OnSemi_CASE100CY"
+	(footprint "forklift_sensor_board:OnSemi_CASE100CY"
 		(layer "F.Cu")
 		(at 100.091 138.297)
@@
 		)
 	)
-	(footprint "HKUST_RDC2024_Footprint_Lib:R_0603_1608Metric"
+	(footprint "forklift_sensor_board:R_0603_1608Metric"
 		(layer "F.Cu")
 		(at 99.123 132.731 -90)
@@
 		)
 	)
-	(footprint "OptoDevice:OnSemi_CASE100CY"
+	(footprint "forklift_sensor_board:OnSemi_CASE100CY"
 		(layer "F.Cu")
 		(at 109.8155 138.297)
@@
 		)
 	)
-	(footprint "OptoDevice:OnSemi_CASE100CY"
+	(footprint "forklift_sensor_board:OnSemi_CASE100CY"
 		(layer "F.Cu")
 		(at 119.54 138.297)
@@
 		)
 	)
-	(footprint "FFC2A32-10-T:GCT_FFC2A32-10-T"
+	(footprint "forklift_sensor_board:GCT_FFC2A32-10-T"
 		(layer "B.Cu")
 		(at 99.86 112.438)
