File: sensor_board/sensor_board.kicad_sch (KiCad schematic)
At the start: 24 parts, among them J2 FFC2A32-10-T, U1 QRE1113GR, U2 QRE1113GR, U3 QRE1113GR, U4 QRE1113GR, U5 QRE1113GR, U6 QRE1113GR, U7 QRE1113GR

Commit message: update lib and step for sensor board
Parts:
- H1, H2: symbol HKUST_RDC2024_Symbol_Lib:MountingHole -> forklift_sensor_board:MountingHole
- J2: symbol FFC2A32-10-T:FFC2A32-10-T -> forklift_sensor_board:FFC2A32-10-T
- R1, R10, R11, R12, R13, R14, R2, R3, R4, R5, R6, R7, R8, R9: symbol HKUST_RDC2024_Symbol_Lib:R_Small_US -> forklift_sensor_board:R_Small_US
- U1, U2, U3, U4, U5, U6, U7: symbol Sensor_Proximity:QRE1113GR -> forklift_sensor_board:QRE1113GR
Changed lines of the file:
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@@
 	)
 	(symbol
-		(lib_id "Sensor_Proximity:QRE1113GR")
+		(lib_id "forklift_sensor_board:QRE1113GR")
 		(at 39.37 82.55 0)
 		(unit 1)
@@
 	)
 	(symbol
-		(lib_id "HKUST_RDC2024_Symbol_Lib:R_Small_US")
+		(lib_id "forklift_sensor_board:R_Small_US")
 		(at 85.09 72.39 0)
 		(unit 1)
@@
 	)
 	(symbol
-		(lib_id "Sensor_Proximity:QRE1113GR")
+		(lib_id "forklift_sensor_board:QRE1113GR")
 		(at 93.98 82.55 0)
 		(unit 1)
@@
 	)
 	(symbol
-		(lib_id "HKUST_RDC2024_Symbol_Lib:R_Small_US")
+		(lib_id "forklift_sensor_board:R_Small_US")
 		(at 214.63 72.39 0)
 		(unit 1)
@@
 	)
 	(symbol
-		(lib_id "Sensor_Proximity:QRE1113GR")
+		(lib_id "forklift_sensor_board:QRE1113GR")
 		(at 121.92 82.55 0)
 		(unit 1)
@@
 	)
 	(symbol
-		(lib_id "HKUST_RDC2024_Symbol_Lib:MountingHole")
+		(lib_id "forklift_sensor_board:MountingHole")
 		(at 198.12 113.03 0)
 		(unit 1)
@@
 	)
 	(symbol
-		(lib_id "Sensor_Proximity:QRE1113GR")
+		(lib_id "forklift_sensor_board:QRE1113GR")
 		(at 205.74 82.55 0)
 		(unit 1)
@@
 	)
 	(symbol
-		(lib_id "Sensor_Proximity:QRE1113GR")
+		(lib_id "forklift_sensor_board:QRE1113GR")
 		(at 148.59 82.55 0)
 		(unit 1)
@@
 	)
 	(symbol
-		(lib_id "HKUST_RDC2024_Symbol_Lib:R_Small_US")
+		(lib_id "forklift_sensor_board:R_Small_US")
 		(at 157.48 72.39 0)
 		(unit 1)
@@
 	)
 	(symbol
-		(lib_id "HKUST_RDC2024_Symbol_Lib:MountingHole")
+		(lib_id "forklift_sensor_board:MountingHole")
 		(at 198.12 120.65 0)
 		(unit 1)
@@
 		)
 		(instances
-			(project ""
+			(project "sensor_board"
 				(path "/7e11bd70-3059-48f0-9e9a-cb12c714f4ee"
 					(reference "H1")
@@
 	)
 	(symbol
-		(lib_id "Sensor_Proximity:QRE1113GR")
+		(lib_id "forklift_sensor_board:QRE1113GR")
 		(at 67.31 82.55 0)
 		(unit 1)
@@
 	)
 	(symbol
-		(lib_id "HKUST_RDC2024_Symbol_Lib:R_Small_US")
+		(lib_id "forklift_sensor_board:R_Small_US")
 		(at 185.42 72.39 0)
 		(unit 1)
@@
 	)
 	(symbol
-		(lib_id "HKUST_RDC2024_Symbol_Lib:R_Small_US")
+		(lib_id "forklift_sensor_board:R_Small_US")
 		(at 102.87 72.39 0)
 		(unit 1)
@@
 	)
 	(symbol
-		(lib_id "HKUST_RDC2024_Symbol_Lib:R_Small_US")
+		(lib_id "forklift_sensor_board:R_Small_US")
 		(at 139.7 72.39 0)
 		(unit 1)
@@
 	)
 	(symbol
-		(lib_id "Sensor_Proximity:QRE1113GR")
+		(lib_id "forklift_sensor_board:QRE1113GR")
 		(at 176.53 82.55 0)
 		(unit 1)
@@
 	)
 	(symbol
-		(lib_id "HKUST_RDC2024_Symbol_Lib:R_Small_US")
+		(lib_id "forklift_sensor_board:R_Small_US")
 		(at 58.42 72.39 0)
 		(unit 1)
@@
 	)
 	(symbol
-		(lib_id "HKUST_RDC2024_Symbol_Lib:R_Small_US")
+		(lib_id "forklift_sensor_board:R_Small_US")
 		(at 48.26 72.39 0)
 		(unit 1)
@@
 	)
 	(symbol
-		(lib_id "HKUST_RDC2024_Symbol_Lib:R_Small_US")
+		(lib_id "forklift_sensor_board:R_Small_US")
 		(at 196.85 72.39 0)
 		(unit 1)
@@
 	)
 	(symbol
-		(lib_id "FFC2A32-10-T:FFC2A32-10-T")
+		(lib_id "forklift_sensor_board:FFC2A32-10-T")
 		(at 127 119.38 0)
 		(unit 1)
@@
 		)
 		(instances
-			(project ""
+			(project "sensor_board"
 				(path "/7e11bd70-3059-48f0-9e9a-cb12c714f4ee"
 					(reference "J2")
@@
 	)
 	(symbol
-		(lib_id "HKUST_RDC2024_Symbol_Lib:R_Small_US")
+		(lib_id "forklift_sensor_board:R_Small_US")
 		(at 130.81 72.39 0)
 		(unit 1)
@@
 	)
 	(symbol
-		(lib_id "HKUST_RDC2024_Symbol_Lib:R_Small_US")
+		(lib_id "forklift_sensor_board:R_Small_US")
 		(at 30.48 72.39 0)
 		(unit 1)
@@
 	)
 	(symbol
-		(lib_id "HKUST_RDC2024_Symbol_Lib:R_Small_US")
+		(lib_id "forklift_sensor_board:R_Small_US")
 		(at 76.2 72.39 0)
 		(unit 1)
@@
 	)
 	(symbol
-		(lib_id "HKUST_RDC2024_Symbol_Lib:R_Small_US")
+		(lib_id "forklift_sensor_board:R_Small_US")
 		(at 113.03 72.39 0)
 		(unit 1)
@@
 	)
 	(symbol
-		(lib_id "HKUST_RDC2024_Symbol_Lib:R_Small_US")
+		(lib_id "forklift_sensor_board:R_Small_US")
 		(at 167.64 72.39 0)
 		(unit 1)
