File: STC_mainboard_2025/STC_mainboard(EM_car)/extention_board.kicad_pcb (KiCad board)
At the start: 2 copper layers, 95.7 x 71.9 mm, 135 parts, among them J1 Conn_01x06, J11 Conn_01x04, J2 Conn_01x06, J3 Conn_01x02, J4 Conn_01x02, J5 Conn_01x05, Q1 S8050, SW1 SW_Push, SW2 SW_Push, SW3 SW_Push, SW4 SW_Push, U1 STC16H40K128_CoreBoard, U2 TPS54360DDA, U3 LM1117-3.3, U4 LM1117-3.3, U5 OPA4197xPW, U6 OPA4197xPW

Commit message: STC mainboard update
Parts:
- 3.3V, 5V, GND: footprint Connector_PinHeader_2.54mm:PinHeader_2x03_P2.54mm_Vertical -> EM_mainboard:PinHeader_2x03_P2.54mm_Vertical
- B1: footprint AI8051U_48P_主板_V1.0:BEEP 9x5.5mm -> EM_mainboard:BEEP 9x5.5mm
- C1, C10, C11, C13, C14, C15, C16, C17, C18, C19, C2, C20, C21, C22, C23, C24, C25, C26, C27, C28, C29, C3, C30, C31, C32, C33, C4, C5, C6, C7, C8: footprint HKUST_RDC2024_Footprint_Lib:C_0603_1608Metric -> EM_mainboard:C_0603_1608Metric
- C9: footprint HKUST_RDC2024_Footprint_Lib:CP_Elec_8x10.5 -> EM_mainboard:CP_Elec_8x10.5
- D1, D10, D11, D12, D13, D14, D15, D16, D17, D18, D19, D20, D5, D6, D7, D8, D9: footprint HKUST_RDC2024_Footprint_Lib:D_SMA -> EM_mainboard:D_SMA
- D2, D3, D4: footprint HKUST_RDC2024_Footprint_Lib:LED_0603_1608Metric_Pad1.05x0.95mm_HandSolder -> EM_mainboard:LED_0603_1608Metric_Pad1.05x0.95mm_HandSolder
- Encoder (x2): footprint AI8051U_48P_主板_V1.0kicad:HDR2X3-M -> EM_mainboard:HDR2X3-M
- G*** (x2): footprint LOGO -> EM_mainboard:LOGO
- H1, H2, H3, H4: footprint HKUST_RDC2024_Footprint_Lib:MountingHole_3.2mm_M3 -> EM_mainboard:MountingHole_3.2mm_M3
- J1, J2: footprint Connector_PinHeader_2.54mm:PinHeader_1x06_P2.54mm_Vertical -> EM_mainboard:PinHeader_1x06_P2.54mm_Vertical
- J11, UART1: footprint Connector_PinHeader_2.54mm:PinHeader_1x04_P2.54mm_Vertical -> EM_mainboard:PinHeader_1x04_P2.54mm_Vertical
- J3: footprint Connector_AMASS:AMASS_XT60-F_1x02_P7.20mm_Vertical -> EM_mainboard:AMASS_XT60-F_1x02_P7.20mm_Vertical
- J4: footprint Connector_PinHeader_2.54mm:PinHeader_1x02_P2.54mm_Vertical -> EM_mainboard:PinHeader_1x02_P2.54mm_Vertical
- J5: footprint Connector_PinSocket_2.54mm:PinSocket_1x05_P2.54mm_Vertical -> EM_mainboard:PinSocket_1x05_P2.54mm_Vertical
- L1: footprint HKUST_RDC2024_Footprint_Lib:L_7.3x7.3_H3.5 -> EM_mainboard:L_7.3x7.3_H3.5
- PSW1: footprint spdtsw:toggle_switch_small -> EM_mainboard:toggle_switch_small
- Q1: footprint AI8051U_48P_主板_V1.0:SOT-23 -> EM_mainboard:SOT-23
- R1, R11, R12, R13, R14, R15, R16, R17, R18, R19, R2, R20, R21, R22, R23, R24, R25, R26, R27, R28, R29, R3, R30, R31, R32, R33, R34, R35, R36, R37, R38, R39, R4, R40, R41, R42, R43, R5, R6, R7, R8, R9: footprint HKUST_RDC2024_Footprint_Lib:R_0603_1608Metric -> EM_mainboard:R_0603_1608Metric
- RV1, RV2, RV3, RV4, RV5, RV6, RV7, RV8: footprint Potentiometer_THT:Potentiometer_Bourns_3296W_Vertical -> EM_mainboard:Potentiometer_Bourns_3296W_Vertical
- SW1, SW2, SW3, SW4: footprint HKUST_RDC2024_Footprint_Lib:SW_Push -> EM_mainboard:SW_Push
- U1: footprint STC32G12K128_CoreBoard:STC16H40K128_CoreBoard -> EM_mainboard:STC16H40K128_CoreBoard
- U2: footprint Package_SO:TI_SO-PowerPAD-8_ThermalVias -> EM_mainboard:TI_SO-PowerPAD-8_ThermalVias
- U3, U4: footprint LM1117-3.3:SOT230 -> EM_mainboard:SOT230
- U5, U6: footprint Package_SO:TSSOP-14_4.4x5mm_P0.65mm -> EM_mainboard:TSSOP-14_4.4x5mm_P0.65mm
- wireless: footprint AI8051U_48P_主板_V1.0kicad:HDR2X4-F -> EM_mainboard:HDR2X4-F
