File: STC_mainboard_2025/STC_mainboard(EM_car)/extention_board.kicad_sch (KiCad schematic)
At the start: 133 parts, among them J1 Conn_01x06, J11 Conn_01x04, J2 Conn_01x06, J3 Conn_01x02, J4 Conn_01x02, J5 Conn_01x05, J7 Conn_02x03_Odd_Even, J8 Conn_02x03_Odd_Even, J9 Conn_02x03_Odd_Even, P1 ${VALUE}, P2 ${VALUE}, P3 ${VALUE}, Q1 ${PARTNUMBER}, SW1 SW_Push, SW2 SW_Push, SW3 SW_Push, SW4 SW_Push, U1 STC16H40K128_CoreBoard, U2 TPS54360DDA, U3 LM1117-3.3, U4 LM1117-3.3, U5 OPA4197xPW, U6 OPA4197xPW

Commit message: STC mainboard update
Parts:
- B1: symbol AI8051U_48P_主板_V1.0:BEEP -> EM_mainboard:BEEP
- C1, C10, C11, C17, C18, C19, C20, C21, C22, C23, C24, C25, C26, C27, C28, C29, C30, C31, C32, C33, C4, C7: symbol HKUST_RDC2024_Symbol_Lib:C_Small -> EM_mainboard:C_Small
- C13, C14, C15, C16: symbol HKUST_RDC2023_Tutorial:C_Small -> EM_mainboard:C_Small
- C2, C3, C5, C6, C8: symbol Device:C_Small -> EM_mainboard:C_Small
- C9: symbol HKUST_RDC2023_Tutorial:CP1_Small -> EM_mainboard:CP1_Small
- D1: symbol Device:D_Schottky -> EM_mainboard:D_Schottky
- D10, D11, D12, D13, D14, D15, D16, D17, D18, D19, D20, D5, D6, D7, D8, D9: symbol HKUST_RDC2024_Symbol_Lib:SS54 -> EM_mainboard:SS54
- D2, D3, D4: symbol HKUST_RDC2024_Symbol_Lib:LED_Small -> EM_mainboard:LED_Small
- H1, H2, H3, H4: symbol HKUST_RDC2024_Symbol_Lib:MountingHole -> EM_mainboard:MountingHole
- J1, J2: symbol Connector_Generic:Conn_01x06 -> EM_mainboard:Conn_01x06
- J11, UART1: symbol Connector_Generic:Conn_01x04 -> EM_mainboard:Conn_01x04
- J3, J4: symbol Connector_Generic:Conn_01x02 -> EM_mainboard:Conn_01x02
- J5: symbol Connector_Generic:Conn_01x05 -> EM_mainboard:Conn_01x05
- J7, J8, J9: symbol Connector_Generic:Conn_02x03_Odd_Even -> EM_mainboard:Conn_02x03_Odd_Even
- L1: symbol Device:L_Small -> EM_mainboard:L_Small
- P1, P3: symbol STC8H&16F&32G_主板_V2.3:Header-D-M 2x3P -> EM_mainboard:Header-D-M 2x3P
- P2: symbol STC8H&16F&32G_主板_V2.3:Header-D-F 2x4P -> EM_mainboard:Header-D-F 2x4P
- PSW1: symbol Switch:SW_SPDT -> EM_mainboard:SW_SPDT
- Q1: symbol AI8051U_48P_主板_V1.0:NPN S8050 -> EM_mainboard:NPN S8050
- R1, R3, R4, R5: symbol Device:R_Small_US -> EM_mainboard:R_Small_US
- R11, R12, R13, R14, R15, R16, R17, R18, R19, R2, R20, R21, R22, R23, R24, R25, R26, R27, R28, R29, R30, R31, R32, R33, R34, R35, R36, R37, R38, R39, R40, R41, R42, R43, R6, R7, R8, R9: symbol HKUST_RDC2024_Symbol_Lib:R_Small_US -> EM_mainboard:R_Small_US
- RV1, RV2, RV3, RV4, RV5, RV6, RV7, RV8: symbol Device:R_Potentiometer -> EM_mainboard:R_Potentiometer
- SW1, SW2, SW3, SW4: symbol HKUST_RDC2023_Tutorial:SW_Push -> EM_mainboard:SW_Push
- U1: symbol STC32G12K128_CoreBoard:STC16H40K128_CoreBoard -> EM_mainboard:STC16H40K128_CoreBoard
- U2: symbol HKUST_RDC2023_Tutorial:TPS54360DDA -> EM_mainboard:TPS54360DDA
- U3, U4: symbol LM1117-3.3:LM1117-3.3 -> EM_mainboard:LM1117-3.3
- U5, U6: symbol Amplifier_Operational:OPA4197xPW -> EM_mainboard:OPA4197xPW
