File: intern/pcb/pcb.kicad_sch (KiCad schematic)
At the start: 33 parts, among them J1 Conn_01x02, J10 Conn_01x04, J11 Conn_01x04, J12 RJ45, J13 Screw_Terminal_01x04, J14 Screw_Terminal_01x04, J15 Screw_Terminal_01x04, J16 Conn_01x04, J2 Conn_01x02, J3 Conn_01x02, J4 Conn_01x02, J5 Conn_01x02, J6 Conn_01x02, J7 Conn_01x02, J8 Conn_01x02, J9 Conn_01x02, U2 STM32F103C8T6, U5 TPS54360DDA, U6 LM1117-3.3

Commit message: finalize intern pcb with gbr
Parts:
- added H1, H2, H3, H4: MountingHole, HKUST_RDC2025_Footprint_Lib:MountingHole_3.2mm_M3, symbol HKUST_RDC2025_Symbol_Lib:MountingHole
Connections:
- net sync_pulse is gone; now on net pps_in: J15.2 (Pin_2)
- net Bl: now also J14.4 (Pin_4); no longer J14.1 (Pin_1)
- net G/: now also J14.3 (Pin_3); no longer J14.2 (Pin_2)
- net O: now also J14.2 (Pin_2); no longer J14.3 (Pin_3)
- net O/: now also J14.1 (Pin_1); no longer J14.4 (Pin_4)
